File: electronics/opensync_prototype/output_ports.kicad_sch (KiCad schematic)
At the start: 0 parts

Commit message: KiCAD backup
Other:
- title: Input Trigger Ports -> Output Ports
Changed lines of the file:
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@@
 	(paper "A4")
 	(title_block
-		(title "Input Trigger Ports")
+		(title "Output Ports")
 		(date "2025-10-31")
 		(rev "0.1")
 		(company "OpenPIV Consortium")
-		(comment 1 "Input ports for external triggers")
+		(comment 1 "Output ports for each output channel")
 	)
 )

Commit message: KiCAD backup
Parts:
- added C? (x4): 100n, symbol Device:C
- added R? (x12): 49.9, symbol Device:R
- added U? (x2): SN74LVC8T245, symbol Logic_LevelTranslator:SN74LVC8T245
Connections:
- new net: R?.1, U?.17 (B5)
- new net: R?.1, U?.14 (B8)
- new net: R?.1, U?.15 (B7)
- new net: R?.1, U?.16 (B6)
- new net: R?.1, U?.18 (B4) (x2)
- new net: R?.1, U?.19 (B3) (x2)
- new net: R?.1, U?.20 (B2) (x2)
- new net: R?.1, U?.21 (B1) (x2)
- new net +3.3V: C?.1, C?.1, U?.1 (V_{CCA}), U?.1 (V_{CCA})
- new net +5V: C?.1, C?.1, U?.23 (V_{CCB}), U?.23 (V_{CCB}), U?.24 (V_{CCB}), U?.24 (V_{CCB})
- new net GND: C?.2, C?.2, C?.2, C?.2, U?.11 (GND), U?.11 (GND), U?.12 (GND), U?.12 (GND), U?.13 (GND), U?.13 (GND)
- new net OUTPUT_1: U?.3 (A1)
- new net OUTPUT_10: U?.4 (A2)
- new net OUTPUT_11: U?.5 (A3)
- new net OUTPUT_12: U?.6 (A4)
- new net OUTPUT_2: U?.4 (A2)
- new net OUTPUT_3: U?.5 (A3)
- new net OUTPUT_4: U?.6 (A4)
- new net OUTPUT_5: U?.7 (A5)
- new net OUTPUT_6: U?.8 (A6)
- new net OUTPUT_7: U?.9 (A7)
- new net OUTPUT_8: U?.10 (A8)
- new net OUTPUT_9: U?.3 (A1)
- no-connect marks 0 -> 8

Commit message: Emergency backup
Parts:
- removed U? (x2): SN74LVC8T245, symbol Logic_LevelTranslator:SN74LVC8T245
- added J10, J11, J12, J13, J14, J15, J16, J5, J6, J7, J8, J9: 66012202111305, 66012202111305:66012202111305, symbol 66012202111305:66012202111305
- added U7, U8: SN74LVC8T245, SN74LVC8T245:TTSOP-24, symbol SN74LVC8T245:SN74LVC8T245
- C26, C27, C28, C29: renamed from C?; footprint (none) -> RP2350_80QFN_minimal:C_0402_1005Metric_small_pads
- R33, R34, R35, R36, R37, R38, R39, R40, R41, R42, R43, R44: renamed from R?; footprint (none) -> Resistor_SMD:R_0402_1005Metric
Connections:
- net +3.3V is gone; now on net +5V: C26.1, C27.1
- net +5V: now also U7.P$1, U8.P$1; no longer C28.1, C29.1
- net GND: now also J10.2, J10.3, J11.2, J11.3, J12.2, J12.3, J13.2, J13.3, J14.2, J14.3, J15.2, J15.3, J16.2, J16.3, J5.2, J5.3, J6.2, J6.3, J7.2, J7.3, J8.2, J8.3, J9.2, J9.3, U7.P$11, U7.P$12, U7.P$13, U7.P$2, U7.P$22, U8.P$11, U8.P$12, U8.P$13, U8.P$18, U8.P$19, U8.P$2, U8.P$20, U8.P$21, U8.P$22, U8.P$3, U8.P$4, U8.P$5, U8.P$6
- net OUTPUT_1: now also U7.P$14
- net OUTPUT_10: now also U8.P$15
- net OUTPUT_11: now also U8.P$16
- net OUTPUT_12: now also U8.P$17
- net OUTPUT_2: now also U7.P$15
- net OUTPUT_3: now also U7.P$16
- net OUTPUT_4: now also U7.P$17
- net OUTPUT_5: now also U7.P$18
- net OUTPUT_6: now also U7.P$19
- net OUTPUT_7: now also U7.P$20
- net OUTPUT_8: now also U7.P$21
- net OUTPUT_9: now also U8.P$14
- net at R37.1: now also U7.P$6
- net at R37.2: now also J9.1
- net at R40.1: now also U7.P$3
- net at R39.1: now also U7.P$4
- net at R38.1: now also U7.P$5
- net at R36.1: now also U7.P$7
- net at R35.1: now also U7.P$8
- net at R34.1: now also U7.P$9
- net at R33.1: now also U7.P$10
- net at R35.2: now also J7.1
- net at R33.2: now also J5.1
- net at R40.2: now also J12.1
- net at R36.2: now also J8.1
- net at R44.1: now also U8.P$7
- net at R43.1: now also U8.P$8
- net at R42.1: now also U8.P$9
- net at R41.1: now also U8.P$10
- net at R41.2: now also J13.1
- net at R42.2: now also J14.1
- net at R43.2: now also J15.1
- net at R34.2: now also J6.1
- net at R39.2: now also J11.1
- net at R44.2: now also J16.1
- net at R38.2: now also J10.1
- new net +3V3: C28.1, C29.1, U7.P$23, U7.P$24, U8.P$23, U8.P$24
- no-connect marks 8 -> 0
Other:
- note added: "IC is upside down for performance and easy grounding"
- moved on the sheet: C26, C27, C28, C29, R33, R34, R35, R36, R37, R38, R39, R40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

Commit message: Backup copy
Parts:
- added R45, R46: 10k, Resistor_SMD:R_0402_1005Metric, symbol Device:R
- renumbered J7 to J10, J6 to J11, J5 to J12, J16 to J13, J15 to J14, J14 to J15, J13 to J16, J12 to J5, J11 to J6, J10 to J7, J9 to J8, J8 to J9, R40 to R33, R39 to R34, R38 to R35, R37 to R36, R36 to R37, R35 to R38, R34 to R39, R33 to R40, R44 to R41, R43 to R42, R42 to R43, R41 to R44
Connections:
- net +3V3: now also U7.P$1, U8.P$1, R45.1, R46.1; no longer U7.P$23, U7.P$24, U8.P$23, U8.P$24
- net +5V: now also U7.P$23, U7.P$24, U8.P$23, U8.P$24; no longer U7.P$1, U8.P$1
- net GND: now also U8.P$10, U8.P$14, U8.P$15, U8.P$16, U8.P$17, U8.P$7, U8.P$8, U8.P$9; no longer U7.P$2, U8.P$18, U8.P$19, U8.P$2, U8.P$20, U8.P$21, U8.P$3, U8.P$4, U8.P$5, U8.P$6
- net OUTPUT_1: now also U7.P$10; no longer U7.P$14
- net OUTPUT_10: now also U8.P$5; no longer U8.P$15
- net OUTPUT_11: now also U8.P$4; no longer U8.P$16
- net OUTPUT_12: now also U8.P$3; no longer U8.P$17
- net OUTPUT_2: now also U7.P$9; no longer U7.P$15
- net OUTPUT_3: now also U7.P$8; no longer U7.P$16
- net OUTPUT_4: now also U7.P$7; no longer U7.P$17
- net OUTPUT_5: now also U7.P$6; no longer U7.P$18
- net OUTPUT_6: now also U7.P$5; no longer U7.P$19
- net OUTPUT_7: now also U7.P$4; no longer U7.P$20
- net OUTPUT_8: now also U7.P$3; no longer U7.P$21
- net OUTPUT_9: now also U8.P$6; no longer U8.P$14
- net at R36.1: now also U7.P$17; no longer U7.P$6
- net at R38.1: now also U7.P$19; no longer U7.P$8
- net at R40.1: now also U7.P$21; no longer U7.P$10
- net at R33.1: now also U7.P$14; no longer U7.P$3
- net at R34.1: now also U7.P$15; no longer U7.P$4
- net at R35.1: now also U7.P$16; no longer U7.P$5
- net at R37.1: now also U7.P$18; no longer U7.P$7
- net at R39.1: now also U7.P$20; no longer U7.P$9
- net at R44.1: now also U8.P$21; no longer U8.P$10
- net at R43.1: now also U8.P$20; no longer U8.P$9
- net at R42.1: now also U8.P$19; no longer U8.P$8
- net at R41.1: now also U8.P$18; no longer U8.P$7
- new net: R45.2, U7.P$2
- new net: R46.2, U8.P$2
Other:
- note removed: "IC is upside down for performance and easy grounding"
- moved on the sheet: C26, C27, C28, C29, U7, U8
