File: electronics/opensync_prototype/opensync_prototype.kicad_pcb (KiCad board)
At the start: 2 copper layers, 3.9 x 4.8 mm, 101 parts, among them J1 61400416121, J10 66012202111305, J11 66012202111305, J12 66012202111305, J13 66012202111305, J14 66012202111305, J15 66012202111305, J16 66012202111305, J2 66012202111305, J3 66012202111305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

Commit message: Backup copy
Parts:
- added R45: 10k, Resistor_SMD:R_0402_1005Metric, F.Cu at (80.5, 122.5)
- added R46: 10k, Resistor_SMD:R_0402_1005Metric, F.Cu at (127.0, 122.5)
- moved J2 140.1 mm to (20.0, 155.0), turned to 180 degrees
- moved J3 137.6 mm to (30.0, 155.0), turned to 180 degrees
- moved J4 135.1 mm to (40.0, 155.0), turned to 180 degrees
- moved U1 107.3 mm to (108.0, 82.3), turned to -90 degrees
- moved R25 96.2 mm to (99.8, 52.0)
- moved Y1 92.4 mm to (100.0, 114.0), turned to 90 degrees
- moved R26 90.4 mm to (101.1, 52.0)
- moved U3 90.2 mm to (103.0, 60.9)
- moved J1 89.6 mm to (103.0, 37.4)
- moved U2 89.0 mm to (100.0, 100.0)
- moved J5 84.2 mm to (50.0, 155.0), turned to 180 degrees
- moved J6 82.7 mm to (60.0, 155.0), turned to 180 degrees
- moved J7 81.3 mm to (70.0, 155.0), turned to 180 degrees
- moved J8 80.1 mm to (80.0, 155.0), turned to 180 degrees
- moved J16 79.6 mm to (160.0, 155.0), turned to 180 degrees
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Connections:
- net /Microcontroller and Ext. Clock/USB_D+ renamed /Power and Data/USB_D+
- net /Microcontroller and Ext. Clock/USB_D- renamed /Power and Data/USB_D-
- U2 pad 1: /Input Ports/TRIGGER_3 -> /Microcontroller and Ext. Clock/CLOCK_1
- U2 pad 11: /Microcontroller and Ext. Clock/OUTPUT_5 -> unconnected-(U2-GPIO12-Pad11)
- U2 pad 12: /Microcontroller and Ext. Clock/OUTPUT_6 -> unconnected-(U2-GPIO13-Pad12)
- U2 pad 13: /Microcontroller and Ext. Clock/OUTPUT_7 -> unconnected-(U2-GPIO14-Pad13)
- U2 pad 14: /Microcontroller and Ext. Clock/OUTPUT_8 -> unconnected-(U2-GPIO15-Pad14)
- U2 pad 16: /Microcontroller and Ext. Clock/OUTPUT_9 -> unconnected-(U2-GPIO16-Pad16)
- U2 pad 17: /Microcontroller and Ext. Clock/OUTPUT_10 -> unconnected-(U2-GPIO17-Pad17)
- U2 pad 18: /Microcontroller and Ext. Clock/OUTPUT_11 -> /Input Ports/TRIGGER_3
- U2 pad 19: /Microcontroller and Ext. Clock/OUTPUT_12 -> /Input Ports/TRIGGER_2
- U2 pad 2: /Input Ports/TRIGGER_2 -> /Microcontroller and Ext. Clock/CLOCK_2
- U2 pad 20: unconnected-(U2-GPIO20-Pad20) -> /Input Ports/TRIGGER_1
- U2 pad 21: unconnected-(U2-GPIO21-Pad21) -> /Microcontroller and Ext. Clock/OUTPUT_1
- U2 pad 22: unconnected-(U2-GPIO22-Pad22) -> /Microcontroller and Ext. Clock/OUTPUT_2
- U2 pad 23: unconnected-(U2-GPIO23-Pad23) -> /Microcontroller and Ext. Clock/OUTPUT_3
- U2 pad 25: unconnected-(U2-GPIO24-Pad25) -> /Microcontroller and Ext. Clock/OUTPUT_4
- U2 pad 26: unconnected-(U2-GPIO25-Pad26) -> /Microcontroller and Ext. Clock/OUTPUT_5
- U2 pad 27: unconnected-(U2-GPIO26-Pad27) -> /Microcontroller and Ext. Clock/OUTPUT_6
- U2 pad 28: unconnected-(U2-GPIO27-Pad28) -> /Microcontroller and Ext. Clock/OUTPUT_7
- U2 pad 3: /Input Ports/TRIGGER_1 -> /Microcontroller and Ext. Clock/CLOCK_3
- U2 pad 36: unconnected-(U2-GPIO28-Pad36) -> /Microcontroller and Ext. Clock/OUTPUT_8
- U2 pad 37: unconnected-(U2-GPIO29-Pad37) -> /Microcontroller and Ext. Clock/OUTPUT_9
- U2 pad 38: unconnected-(U2-GPIO30-Pad38) -> /Microcontroller and Ext. Clock/OUTPUT_10
- U2 pad 39: unconnected-(U2-GPIO31-Pad39) -> /Microcontroller and Ext. Clock/OUTPUT_11
- U2 pad 40: unconnected-(U2-GPIO32-Pad40) -> /Microcontroller and Ext. Clock/OUTPUT_12
- U2 pad 6: /Microcontroller and Ext. Clock/OUTPUT_1 -> unconnected-(U2-GPIO8-Pad6)
- U2 pad 7: /Microcontroller and Ext. Clock/OUTPUT_2 -> unconnected-(U2-GPIO9-Pad7)
- U2 pad 77: /Microcontroller and Ext. Clock/CLOCK_1 -> unconnected-(U2-GPIO0-Pad77)
- U2 pad 78: /Microcontroller and Ext. Clock/CLOCK_2 -> unconnected-(U2-GPIO1-Pad78)
- U2 pad 79: /Microcontroller and Ext. Clock/CLOCK_3 -> unconnected-(U2-GPIO2-Pad79)
- U2 pad 8: /Microcontroller and Ext. Clock/OUTPUT_3 -> unconnected-(U2-GPIO10-Pad8)
- U2 pad 9: /Microcontroller and Ext. Clock/OUTPUT_4 -> unconnected-(U2-GPIO11-Pad9)
- U7 pad P$1: +5V -> +3V3
- U7 pad P$10: Net-(R33-Pad1) -> /Microcontroller and Ext. Clock/OUTPUT_1
- U7 pad P$14: /Microcontroller and Ext. Clock/OUTPUT_1 -> Net-(R33-Pad1)
- U7 pad P$15: /Microcontroller and Ext. Clock/OUTPUT_2 -> Net-(R34-Pad1)
- U7 pad P$16: /Microcontroller and Ext. Clock/OUTPUT_3 -> Net-(R35-Pad1)
- U7 pad P$17: /Microcontroller and Ext. Clock/OUTPUT_4 -> Net-(R36-Pad1)
- U7 pad P$18: /Microcontroller and Ext. Clock/OUTPUT_5 -> Net-(R37-Pad1)
- U7 pad P$19: /Microcontroller and Ext. Clock/OUTPUT_6 -> Net-(R38-Pad1)
- U7 pad P$2: GND -> Net-(R45-Pad2)
- U7 pad P$20: /Microcontroller and Ext. Clock/OUTPUT_7 -> Net-(R39-Pad1)
- U7 pad P$21: /Microcontroller and Ext. Clock/OUTPUT_8 -> Net-(R40-Pad1)
- U7 pad P$23: +3V3 -> +5V
- U7 pad P$24: +3V3 -> +5V
- U7 pad P$3: Net-(R40-Pad1) -> /Microcontroller and Ext. Clock/OUTPUT_8
- U7 pad P$4: Net-(R39-Pad1) -> /Microcontroller and Ext. Clock/OUTPUT_7
- U7 pad P$5: Net-(R38-Pad1) -> /Microcontroller and Ext. Clock/OUTPUT_6
- U7 pad P$6: Net-(R37-Pad1) -> /Microcontroller and Ext. Clock/OUTPUT_5
- U7 pad P$7: Net-(R36-Pad1) -> /Microcontroller and Ext. Clock/OUTPUT_4
- U7 pad P$8: Net-(R35-Pad1) -> /Microcontroller and Ext. Clock/OUTPUT_3
- U7 pad P$9: Net-(R34-Pad1) -> /Microcontroller and Ext. Clock/OUTPUT_2
- U8 pad P$1: +5V -> +3V3
- U8 pad P$10: Net-(R41-Pad1) -> GND
- U8 pad P$14: /Microcontroller and Ext. Clock/OUTPUT_9 -> GND
- U8 pad P$15: /Microcontroller and Ext. Clock/OUTPUT_10 -> GND
- U8 pad P$16: /Microcontroller and Ext. Clock/OUTPUT_11 -> GND
- U8 pad P$17: /Microcontroller and Ext. Clock/OUTPUT_12 -> GND
- U8 pad P$18: GND -> Net-(R41-Pad1)
- U8 pad P$19: GND -> Net-(R42-Pad1)
- U8 pad P$2: GND -> Net-(R46-Pad2)
- U8 pad P$20: GND -> Net-(R43-Pad1)
- U8 pad P$21: GND -> Net-(R44-Pad1)
- U8 pad P$23: +3V3 -> +5V
- U8 pad P$24: +3V3 -> +5V
- U8 pad P$3: GND -> /Microcontroller and Ext. Clock/OUTPUT_12
- U8 pad P$4: GND -> /Microcontroller and Ext. Clock/OUTPUT_11
- U8 pad P$5: GND -> /Microcontroller and Ext. Clock/OUTPUT_10
- U8 pad P$6: GND -> /Microcontroller and Ext. Clock/OUTPUT_9
- U8 pad P$7: Net-(R44-Pad1) -> GND
- U8 pad P$8: Net-(R43-Pad1) -> GND
- U8 pad P$9: Net-(R42-Pad1) -> GND
Other:
- outline, holes or cut-outs redrawn

Commit message: Emergency backup
Parts:
- moved U6 64.5 mm to (52.0, 119.5)
- moved U5 57.8 mm to (53.5, 108.8)
- moved R14 53.5 mm to (74.5, 120.5), turned to 180 degrees
- moved R15 50.5 mm to (75.0, 119.5)
- moved U4 49.9 mm to (51.5, 97.3)
- moved R16 47.5 mm to (75.5, 118.5)
- moved C18 47.3 mm to (83.0, 54.1)
- moved C20 47.3 mm to (83.0, 58.1)
- moved C22 47.3 mm to (83.0, 62.0)
- moved C27 46.5 mm to (128.0, 131.5)
- moved C28 46.5 mm to (81.5, 121.5)
- moved R17 44.6 mm to (76.0, 117.5)
- moved R13 42.6 mm to (74.0, 121.5)
- moved R7 40.7 mm to (90.0, 103.0), turned to 90 degrees
- moved R8 38.6 mm to (88.5, 103.5), turned to 90 degrees
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Connections:
- net /Input Ports/TRIGGER_1 renamed /Microcontroller and Ext. Clock/TRIGGER_3
- net /Input Ports/TRIGGER_2 renamed /Microcontroller and Ext. Clock/TRIGGER_2
- net /Input Ports/TRIGGER_3 renamed /Microcontroller and Ext. Clock/TRIGGER_1
Other:
- outline, holes or cut-outs redrawn
