File: electronics/opensync_prototype/_autosave-opensync_prototype.kicad_pcb (KiCad board)
At the start: 4 copper layers, 160 x 100 mm, 143 parts, among them J1 61400416121, J10 66012202111305, J11 66012202111305, J12 66012202111305, J13 66012202111305, J14 66012202111305, J15 66012202111305, J16 66012202111305, J2 66012202111305, J3 66012202111305, J4 66012202111305, J5 66012202111305, J6 66012202111305, J7 66012202111305, J8 66012202111305, J9 66012202111305, SW1 SW_Push, SW2 SW_Push, U1 NCP1117-3.3_SOT223, U10 SN74LVC1T45DCKR, U11 SN74LVC1T45DCKR, U12 SN74LVC1T45DCKR, U13 SN74LVC1T45DCKR, U14 SN74LVC1T45DCKR, U15 SN74LVC1T45DCKR, U16 SN74LVC1T45DCKR, U17 SN74LVC1T45DCKR, U18 SN74LVC1T45DCKR, U19 SN74LVC1T45DCKR, U2 RP2354_80QFN, U3 ADUM4160, U4 SN74LVC1G17DCKR, U5 SN74LVC1G17DCKR, U6 SN74LVC1G17DCKR, U8 SN74LVC1T45DCKR, U9 SN74LVC1T45DCKR, Y1 ABM8-272-T3

Commit message: Backup
Parts:
- moved C23 66.5 mm to (139.0, 67.0)
- moved C24 66.5 mm to (139.0, 69.0)
- moved C25 66.5 mm to (139.0, 70.9)
- moved U4 55.5 mm to (70.5, 128.0), turned to 90 degrees
- moved R27 48.1 mm to (71.0, 133.5)
- moved R28 44.0 mm to (81.5, 133.0)
- moved R29 43.2 mm to (91.5, 133.5)
- moved U5 41.1 mm to (81.2, 128.0), turned to 90 degrees
- moved R30 40.6 mm to (70.5, 131.5), turned to 90 degrees
- moved R31 36.1 mm to (81.0, 131.0), turned to 90 degrees
- moved R32 35.3 mm to (91.0, 131.5), turned to 90 degrees
- moved R25 27.5 mm to (156.0, 64.0)
- moved R26 27.3 mm to (157.5, 64.0)
- moved R3 26.4 mm to (117.2, 85.2)
- moved C18 26.4 mm to (123.5, 73.8)
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