File: electronics/opensync_prototype/input_ports.kicad_sch (KiCad schematic)
At the start: 12 parts

Commit message: Emergency backup
Parts:
- added J2, J3, J4: 66012202111305, 66012202111305:66012202111305, symbol 66012202111305:66012202111305
- C23, C24, C25: renamed from C?; footprint (none) -> RP2350_80QFN_minimal:C_0402_1005Metric_small_pads
- R27, R28, R29, R30, R31, R32: renamed from R?; footprint (none) -> Resistor_SMD:R_0402_1005Metric
- gave numbers to parts that had none: 3
Connections:
- net GND: now also J2.2, J2.3, J3.2, J3.3, J4.2, J4.3
- net at R29.1, R32.1: now also J4.1
- net at R28.1, R31.1: now also J3.1
- net at R27.1, R30.1: now also J2.1

Commit message: Updated PCB design
Parts:
- removed C24, C25: 100n, RP2350_80QFN_minimal:C_0402_1005Metric_small_pads, symbol Device:C
- removed J2, J3, J4: 66012202111305, 66012202111305:66012202111305, symbol 66012202111305:66012202111305
- removed R28, R29: 47k, Resistor_SMD:R_0402_1005Metric, symbol Device:R
- removed R31, R32: 470, Resistor_SMD:R_0402_1005Metric, symbol Device:R
- removed U5, U6: SN74LVC1G17DCKR, SN74LVC1G17DCKR:SOT65P210X110-5N, symbol SN74LVC1G17DCKR:SN74LVC1G17DCKR
- added J2: 61611042121502, 61611042121502:61611042121502, symbol 61611042121502:61611042121502
- renumbered R30 to R13
Connections:
- net GND: now also J2.2, J2.3, J2.4, J2.5
- net at R13.1, R27.1: now also J2.1
Other:
- title: Input Trigger Ports -> OpenSync Input Trigger Ports
