File: electronics/opensync_prototype/opensync_prototype.kicad_sch (KiCad schematic)
At the start: 0 parts

Commit message: Backup push
Other:
- added sheet Power and Data (usb_connection.kicad_sch)
Changed lines of the file:
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@@
+		)
+	)
+	(sheet
+		(at 54.61 66.04)
+		(size 45.72 27.94)
+		(exclude_from_sim no)
+		(in_bom yes)
+		(on_board yes)
+		(dnp no)
+		(fields_autoplaced yes)
+		(stroke
+			(width 0.1524)
+			(type solid)
+		)
+		(fill
+			(color 0 0 0 0.0000)
+		)
+		(property "Sheetname" "Power and Data"
+			(at 54.61 65.3284 0)
+			(effects
+				(font
+					(size 1.27 1.27)
+				)
+				(justify left bottom)
+			)
+		)
+		(property "Sheetfile" "usb_connection.kicad_sch"
+			(at 54.61 94.5646 0)
+			(effects
+				(font
+					(size 1.27 1.27)
+				)
+				(justify left top)
+			)
+		)
+		(instances
+			(project "opensync_prototype"
+				(path "/97d97b34-a2f9-4e5e-9870-299ade25a4f4"
+					(page "3")
+				)
+			)
 		)
 	)

Commit message: KiCAD backup
Other:
- added sheet Input Ports (input_ports.kicad_sch)
- added sheet Output Ports (output_ports.kicad_sch)
Changed lines of the file:
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@@
+	)
+	(sheet
+		(at 157.48 102.87)
+		(size 44.45 27.94)
+		(exclude_from_sim no)
+		(in_bom yes)
+		(on_board yes)
+		(dnp no)
+		(fields_autoplaced yes)
+		(stroke
+			(width 0.1524)
+			(type solid)
+		)
+		(fill
+			(color 0 0 0 0.0000)
+		)
+		(property "Sheetname" "Output Ports"
+			(at 157.48 102.1584 0)
+			(effects
+				(font
+					(size 1.27 1.27)
+				)
+				(justify left bottom)
+			)
+		)
+		(property "Sheetfile" "output_ports.kicad_sch"
+			(at 157.48 131.3946 0)
+			(effects
+				(font
+					(size 1.27 1.27)
+				)
+				(justify left top)
+			)
+		)
+		(instances
+			(project "opensync_prototype"
+				(path "/97d97b34-a2f9-4e5e-9870-299ade25a4f4"
+					(page "5")
+				)
+			)
+		)
 	)
 	(sheet
@@
 				)
 			)
+		)
+	)
+	(sheet
+		(at 157.48 66.04)
+		(size 44.45 27.94)
+		(exclude_from_sim no)
+		(in_bom yes)
+		(on_board yes)
+		(dnp no)
+		(fields_autoplaced yes)
+		(stroke
+			(width 0.1524)
+			(type solid)
+		)
+		(fill
+			(color 0 0 0 0.0000)
+		)
+		(property "Sheetname" "Input Ports"
+			(at 157.48 65.3284 0)
+			(effects
+				(font
+					(size 1.27 1.27)
+				)
+				(justify left bottom)
+			)
+		)
+		(property "Sheetfile" "input_ports.kicad_sch"
+			(at 157.48 94.5646 0)
+			(effects
+				(font
+					(size 1.27 1.27)
+				)
+				(justify left top)
+			)
+		)
+		(instances
+			(project "opensync_prototype"
+				(path "/97d97b34-a2f9-4e5e-9870-299ade25a4f4"
+					(page "4")
+				)
+			)

Commit message: Emergency backup
Other:
- sheet Input Ports ports: added TRIGGER_1, TRIGGER_2, TRIGGER_3; removed none
- sheet Microcontroller and Ext. Clock ports: added OUTPUT_1, OUTPUT_10, OUTPUT_11, OUTPUT_12, OUTPUT_2, OUTPUT_3, OUTPUT_4, OUTPUT_5, OUTPUT_6, OUTPUT_7, OUTPUT_8, OUTPUT_9, TRIGGER_1, TRIGGER_2, TRIGGER_3, USB_D+, USB_D-; removed none
- sheet Output Ports ports: added OUTPUT_1, OUTPUT_10, OUTPUT_11, OUTPUT_12, OUTPUT_2, OUTPUT_3, OUTPUT_4, OUTPUT_5, OUTPUT_6, OUTPUT_7, OUTPUT_8, OUTPUT_9; removed none
- sheet Power and Data ports: added USB_D+, USB_D-; removed none

Commit message: Backup
Other:
- removed sheet Output Ports
- added sheet Output Ports 1 to 3 (output_ports_1_to_3.kicad_sch)
- added sheet Output Ports 10 to 12 (output_ports_10_to_12.kicad_sch)
- added sheet Output Ports 4 to 6 (output_ports_4_to_6.kicad_sch)
- added sheet Output Ports 7 to 9 (output_ports_7_to_9.kicad_sch)

Commit message: Updated PCB design
Other:
- removed sheet Output Ports 1 to 3
- removed sheet Output Ports 10 to 12
- removed sheet Output Ports 4 to 6
- removed sheet Output Ports 7 to 9
- added sheet Mounting Holes (mount_holes.kicad_sch)
- added sheet Output Ports 1 to 4 (output_ports_1_to_4.kicad_sch)
- added sheet Output Ports 5 to 8 (output_ports_5_to_8.kicad_sch)
- sheet Input Ports ports: added none; removed TRIGGER_2, TRIGGER_3
- sheet Microcontroller and Ext. Clock ports: added none; removed OUTPUT_10, OUTPUT_11, OUTPUT_12, OUTPUT_9, TRIGGER_2, TRIGGER_3
- note added: "Output Ports 9 to 16 will go Here Once Designed"
