File: electronics/opensync_prototype/output_ports_1_to_4.kicad_sch (KiCad schematic)
At the start: 24 parts, among them J4 61611042121502, J5 61611042121502, J6 61611042121502, J7 61611042121502, U5 SN74LVC1T45DCKR, U6 SN74LVC1T45DCKR, U7 SN74LVC1T45DCKR, U8 SN74LVC1T45DCKR

Commit message: GFround and power plane rework
Changed lines of the file:
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@@
 	(wire
 		(pts
+			(xy 223.52 76.2) (xy 223.52 80.01)
+		)
+		(stroke
+			(width 0)
+			(type default)
+		)
+	)
+	(wire
+		(pts
 			(xy 170.18 151.13) (xy 171.45 151.13)
 		)
@@
 	(wire
 		(pts
-			(xy 223.52 77.47) (xy 223.52 80.01)
-		)
-		(stroke
-			(width 0)
-			(type default)
-		)
-	)
-	(wire
-		(pts
 			(xy 77.47 87.63) (xy 80.01 87.63)
 		)
@@
 	(symbol
 		(lib_id "power:GND")
-		(at 223.52 77.47 180)
+		(at 223.52 76.2 180)
 		(unit 1)
 		(exclude_from_sim no)
@@
 		(fields_autoplaced yes)
 		(property "Reference" "#PWR024"
-			(at 223.52 71.12 0)
+			(at 223.52 69.85 0)
 			(effects
 				(font
@@
 		)
 		(property "Value" "GND"
-			(at 223.52 72.39 0)
+			(at 223.52 71.12 0)
 			(effects
 				(font
@@
 		)
 		(property "Footprint" ""
-			(at 223.52 77.47 0)
+			(at 223.52 76.2 0)
 			(effects
 				(font
@@
 		)
 		(property "Datasheet" ""
-			(at 223.52 77.47 0)
+			(at 223.52 76.2 0)
 			(effects
 				(font
@@
 		)
 		(property "Description" "Power symbol creates a global label with name \"GND\" , ground"
-			(at 223.52 77.47 0)
+			(at 223.52 76.2 0)
 			(effects
 				(font
