File: electronics/opensync_prototype/microcontroller_and_clock.kicad_sch (KiCad schematic)
At the start: 40 parts, among them SW1 SW_Push, SW2 SW_Push, U2 RP2354_80QFN, Y1 ABM8-272-T3

Commit message: PCB touch-ups
Connections:
- net QSPI_SD3: now reaches U2.70 (QSPI_SD3)
- net QSPI_SCLK: now reaches U2.71 (QSPI_SCLK)
- net QSPI_SD0: now reaches U2.72 (QSPI_SD0)
- net QSPI_SD2: now reaches U2.73 (QSPI_SD2)
- net QSPI_SD1: now reaches U2.74 (QSPI_SD1)
- net QSPL_SS renamed QSPI_SS
Changed lines of the file:
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@@
-	)
-	(no_connect
-		(at 102.87 69.85)
 	)
 	(no_connect
@@
 	)
 	(no_connect
-		(at 102.87 72.39)
-	)
-	(no_connect
 		(at 171.45 82.55)
 	)
@@
 	)
 	(no_connect
+		(at 92.71 76.2)
+	)
+	(no_connect
 		(at 171.45 138.43)
 	)
@@
 	)
 	(no_connect
+		(at 92.71 64.77)
+	)
+	(no_connect
 		(at 171.45 163.83)
 	)
@@
 	)
 	(no_connect
-		(at 102.87 67.31)
-	)
-	(no_connect
 		(at 102.87 114.3)
 	)
@@
 	)
 	(no_connect
+		(at 92.71 72.39)
+	)
+	(no_connect
 		(at 171.45 110.49)
 	)
 	(no_connect
+		(at 92.71 67.31)
+	)
+	(no_connect
 		(at 171.45 59.69)
 	)
@@
 	)
 	(no_connect
-		(at 102.87 64.77)
-	)
-	(no_connect
 		(at 171.45 158.75)
 	)
 	(no_connect
+		(at 92.71 69.85)
+	)
+	(no_connect
 		(at 171.45 85.09)
 	)
@@
 	)
 	(no_connect
-		(at 102.87 76.2)
-	)
-	(no_connect
 		(at 171.45 140.97)
 	)
@@
 	(wire
 		(pts
+			(xy 92.71 69.85) (xy 102.87 69.85)
+		)
+		(stroke
+			(width 0)
+			(type default)
+		)
+	)
+	(wire
+		(pts
 			(xy 135.89 24.13) (xy 138.43 24.13)
 		)
@@
 	(wire
 		(pts
+			(xy 92.71 72.39) (xy 102.87 72.39)
+		)
+		(stroke
+			(width 0)
+			(type default)
+		)
+	)
+	(wire
+		(pts
 			(xy 54.61 27.94) (xy 62.23 27.94)
 		)
@@
 	(wire
 		(pts
+			(xy 92.71 76.2) (xy 102.87 76.2)
+		)
+		(stroke
+			(width 0)
+			(type default)
+		)
+	)
+	(wire
+		(pts
 			(xy 72.39 27.94) (xy 72.39 43.18)
 		)
@@
 	(wire
 		(pts
+			(xy 92.71 67.31) (xy 102.87 67.31)
+		)
+		(stroke
+			(width 0)
+			(type default)
+		)
+	)
+	(wire
+		(pts
 			(xy 173.99 24.13) (xy 185.42 24.13)
 		)
@@
 		(pts
 			(xy 247.65 144.78) (xy 247.65 148.59)
+		)
+		(stroke
+			(width 0)
+			(type default)
+		)
+	)
+	(wire
+		(pts
+			(xy 92.71 64.77) (xy 102.87 64.77)
 		)
 		(stroke
@@
 		)
 	)
-	(label "QSPL_SS"
+	(label "QSPI_SS"
 		(at 92.71 60.96 0)
 		(effects
@@
 		)
 	)
+	(label "QSPI_SD0"
+		(at 92.71 64.77 0)
+		(effects
+			(font
+				(size 1.27 1.27)
+			)
+			(justify left bottom)
+		)
+	)
+	(label "QSPI_SCLK"
+		(at 92.71 76.2 0)
+		(effects
+			(font
+				(size 1.27 1.27)
+			)
+			(justify left bottom)
+		)
+	)
 	(label "CLOCK_3"
 		(at 171.45 57.15 0)
@@
 		)
 	)
+	(label "QSPI_SD3"
+		(at 92.71 72.39 0)
+		(effects
+			(font
+				(size 1.27 1.27)
+			)
+			(justify left bottom)
+		)
+	)
+	(label "QSPI_SD1"
+		(at 92.71 67.31 0)
+		(effects
+			(font
+				(size 1.27 1.27)
+			)
+			(justify left bottom)
+		)
+	)
 	(label "VREG_LX"
 		(at 93.98 50.8 0)
@@
 		(effects
 			(font
+				(size 1.27 1.27)
+			)
+			(justify left bottom)
+		)
+	)
+	(label "QSPI_SD2"
+		(at 92.71 69.85 0)
+		(effects
+			(font

Commit message: Refined PCB
Parts:
- added D1, D2: LED, LED_SMD:LED_0603_1608Metric, symbol Device:LED
- added J12: SM03B-SRSS-TB, Connector_JST:JST_SH_SM03B-SRSS-TB_1x03-1MP_P1.00mm_Horizontal, symbol Connector_Generic_MountingPin:Conn_01x03_MountingPin
- added J13: 61611042121502, 61611042121502:61611042121502, symbol 61611042121502:61611042121502
- added R14: 100, Resistor_SMD:R_0402_1005Metric, symbol Device:R
- added R8: 47k, Resistor_SMD:R_0402_1005Metric, symbol Device:R
- added R9: 169, Resistor_SMD:R_0402_1005Metric, symbol Device:R
Connections:
- net +3V3: now also R8.1
- net GND: now also J12.2 (Pin_2), J12.MP (MountPin), J13.2, J13.3, J13.4, J13.5, R14.1, R9.1
- net SWCLK: now reaches U2.33 (SWCLK)
- net SWCLK: now also J12.1 (Pin_1)
- net SWD: now reaches U2.34 (SWD)
- net SWD: now also J12.3 (Pin_3)
- net OUTPUT_9: now reaches U2.42 (GPIO33)
- net OUTPUT_10: now reaches U2.43 (GPIO34)
- net OUTPUT_11: now reaches U2.44 (GPIO35)
- net OUTPUT_12: now reaches U2.45 (GPIO36)
- net OUTPUT_13: now reaches U2.46 (GPIO37)
- net OUTPUT_14: now reaches U2.47 (GPIO38)
- net OUTPUT_15: now reaches U2.48 (GPIO39)
- net OUTPUT_16: now reaches U2.49 (GPIO40_ADC0)
- net ERROR_LED: now reaches U2.54 (GPIO43_ADC3)
- net ERROR_LED: now also D2.2 (A)
- net SAFETY_INTERLOCK: now reaches U2.55 (GPIO44_ADC4)
- net SAFETY_INTERLOCK: now also J13.1, R8.2
- new net: D1.1 (K), R9.2
- new net: D2.1 (K), R14.2
- new net +5V: D1.2 (A)
- no-connect marks 43 -> 39
Other:
- note added: "Error Indicator LED"
- note added: "JST Debug Connector"
- note added: "Power Indicator LED"
- note added: "Safety Interlock"
- moved on the sheet: C2, C3, R2, Y1
