File: electronics/opensync_prototype/usb_connection.kicad_sch (KiCad schematic)
At the start: 4 parts

Commit message: KiCAD backup
Parts:
- added C? (x2): 100n, symbol Device:C
- added R? (x2): 24, symbol Device:R
- added U?: ADUM4160, Package_SO:SOIC-16W_7.5x10.3mm_P1.27mm, symbol Interface_USB:ADUM4160
Connections:
- net GND: now also C?.2, U?.15 (GND2), U?.9 (GND2); no longer C?.2, J?.4 (GND), J?.SH1 (SHIELD), J?.SH2 (SHIELD)
- net USB_D+: now also U?.10 (DD+); no longer J?.3 (D+)
- net USB_D-: now also U?.11 (DD-); no longer J?.2 (D-)
- net VBUS: now also U?.1 (VBUS1); no longer U?.3 (VI)
- new net: J?.3 (D+), R?.1
- new net: R?.2, U?.7 (UD+)
- new net: J?.2 (D-), R?.1
- new net: C?.1, U?.12 (PIN), U?.13 (SPD), U?.14 (VDD2)
- new net: C?.2, U?.3 (VDD1), U?.4 (PDEN), U?.5 (SPU)
- new net: R?.2, U?.6 (UD-)
- new net +5V: U?.16 (VBUS2), U?.3 (VI)
- new net GND_BUS: C?.1, C?.2, J?.4 (GND), J?.SH1 (SHIELD), J?.SH2 (SHIELD), U?.2 (GND1), U?.8 (GND1)
Other:
- moved on the sheet: C?, U?

Commit message: KiCAD backup
Parts:
- added C?: 10u, symbol Device:C
Connections:
- net +5V: now also C?.1
- net GND: now also C?.2
Other:
- moved on the sheet: C?, J?, R?, U?

Commit message: Emergency backup
Parts:
- removed J?: 61729-0010BLF, 61729-0010BLF:AMPHENOL_61729-0010BLF, symbol 61729-0010BLF:61729-0010BLF
- added J1: 61400416121, 61400416121:61400416121, symbol 61400416121:61400416121
- C18, C19, C20, C21, C22: renamed from C?; footprint (none) -> RP2350_80QFN_minimal:C_0402_1005Metric_small_pads
- R25, R26: renamed from R?; footprint (none) -> Resistor_SMD:R_0402_1005Metric
- gave numbers to parts that had none: 2
Connections:
- net GND_BUS: now also J1.4 (GND), J1.S1, J1.S2
- net VBUS: now also J1.1 (VBUS)
- net at R25.1: now also J1.3 (D+)
- net at R26.1: now also J1.2 (D-)

Commit message: Backup copy
Changed lines of the file:
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@@
+		)
+	)
+	(label "USB_D-"
+		(at 87.63 67.31 0)
+		(effects
+			(font
+				(size 1.27 1.27)
+			)
+			(justify left bottom)
+		)
+	)
+	(label "USB_D+"
+		(at 87.63 64.77 0)
+		(effects
+			(font
+				(size 1.27 1.27)
+			)
+			(justify left bottom)
 		)
 	)

Commit message: Updated PCB design
Parts:
- R25, R26: value 24 -> 27
Changed lines of the file:
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@@
 			)
 		)
-		(property "Value" "24"
+		(property "Value" "27"
 			(at 105.41 62.23 90)
 			(effects
@@
 			)
 		)
-		(property "Value" "24"
+		(property "Value" "27"
 			(at 105.664 67.31 90)
 			(effects

Commit message: GFround and power plane rework
Parts:
- removed R25, R26: 27, Resistor_SMD:R_0402_1005Metric, symbol Device:R
- removed U3: ADUM4160, Package_SO:SOIC-16W_7.5x10.3mm_P1.27mm, symbol Interface_USB:ADUM4160
- added L2: 15u, RP2350_80QFN_minimal:L_pol_2016, symbol Device:L
- added L3: 22u, RP2350_80QFN_minimal:L_pol_2016, symbol Device:L
- added U3: NXE2S0505MC, Converter_DCDC:Converter_DCDC_Murata_NXExSxxxxMC_SMD, symbol Regulator_Switching:NXE2S0505MC
- C20: value 100n -> 4.7u
- C22: value 100n -> 10u
Connections:
- net +5V: now also C22.1, L3.2
- net GND: now also U3.7 (-VOUT)
- net GND_BUS: now also U3.1 (-VIN)
- net USB_D+: now also J1.3 (D+)
- net USB_D-: now also J1.2 (D-)
- net VBUS: now also C20.2, L2.1
- new net: L2.2, U3.3 (+VIN)
- new net: L3.1, U3.8 (+VOUT)
Other:
- moved on the sheet: C19, C20, C21, C22, U1

Commit message: Refined PCB
Changed lines of the file:
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@@
+	)
+	(junction
+		(at 92.71 72.39)
+		(diameter 0)
+		(color 0 0 0 0)
 	)
 	(junction
@@
 	)
 	(junction
-		(at 92.71 72.39)
-		(diameter 0)
-		(color 0 0 0 0)
-	)
-	(junction
 		(at 158.75 92.71)
 		(diameter 0)
@@
 	(wire
 		(pts
+			(xy 92.71 72.39) (xy 92.71 82.55)
+		)
+		(stroke
+			(width 0)
+			(type default)
+		)
+	)
+	(wire
+		(pts
 			(xy 97.79 64.77) (xy 97.79 62.23)
 		)
@@
 	(wire
 		(pts
-			(xy 92.71 72.39) (xy 92.71 82.55)
-		)
-		(stroke
-			(width 0)
-			(type default)
-		)
-	)
-	(wire
-		(pts
 			(xy 160.02 74.93) (xy 160.02 73.66)
 		)
@@
 	)
 	(label "USB_D-"
-		(at 87.63 67.31 0)
+		(at 88.9 67.31 0)
 		(effects
 			(font
@@
 	)
 	(label "USB_D+"
-		(at 87.63 64.77 0)
+		(at 88.9 64.77 0)
 		(effects
 			(font
