File: electronics/prototypes/opensync_prototype_4ch/usb_connection.kicad_sch (KiCad schematic)
At the start: 10 parts, among them J1 61400416121, U1 NCP1117-3.3_SOT223, U3 NXE2S0505MC

Commit message: Added part numbers
Parts:
- C18, C19, C21, C22: LCSC (none) -> C1856484
- C20: LCSC (none) -> C326586
- L2: footprint RP2350_80QFN_minimal:L_pol_2016 -> ASPI-4030S-150M-T:IND_ASPI-4030S-150M-T; LCSC (none) -> C5570254
- L3: footprint RP2350_80QFN_minimal:L_pol_2016 -> ASPI6045S220MT:IND_ASPI6045S220MT; LCSC (none) -> C187454
- U1: LCSC (none) -> C26537
Changed lines of the file:
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@@
 			)
 		)
-		(property "Footprint" "RP2350_80QFN_minimal:L_pol_2016"
+		(property "Footprint" "ASPI-4030S-150M-T:IND_ASPI-4030S-150M-T"
 			(at 156.21 63.5 0)
 			(effects
@@
 		)
 		(property "Description" "Inductor"
+			(at 156.21 63.5 0)
+			(effects
+				(font
+					(size 1.27 1.27)
+				)
+				(hide yes)
+			)
+		)
+		(property "LCSC" "C5570254 "
 			(at 156.21 63.5 0)
 			(effects
@@
 			)
 		)
+		(property "LCSC" ""
+			(at 78.74 67.31 0)
+			(effects
+				(font
+					(size 1.27 1.27)
+				)
+			)
+		)
 		(pin "4"
 		)
@@
 			)
 		)
-		(property "Footprint" "RP2350_80QFN_minimal:L_pol_2016"
+		(property "Footprint" "ASPI6045S220MT:IND_ASPI6045S220MT"
 			(at 191.77 63.5 0)
 			(effects
@@
 		)
 		(property "Description" "Inductor"
+			(at 191.77 63.5 0)
+			(effects
+				(font
+					(size 1.27 1.27)
+				)
+				(hide yes)
+			)
+		)
+		(property "LCSC" "C187454"
 			(at 191.77 63.5 0)
 			(effects
@@
 			)
 		)
+		(property "LCSC" "C1856484"
+			(at 185.42 96.52 0)
+			(effects
+				(font
+					(size 1.27 1.27)
+				)
+				(hide yes)
+			)
+		)
 		(pin "1"
 		)
@@
 			)
 		)
+		(property "LCSC" "C26537"
+			(at 172.72 92.71 0)
+			(effects
+				(font
+					(size 1.27 1.27)
+				)
+				(hide yes)
+			)
+		)
 		(pin "2"
 		)
@@
 		)
 		(property "Description" "Unpolarized capacitor"
+			(at 201.93 71.12 0)
+			(effects
+				(font
+					(size 1.27 1.27)
+				)
+				(hide yes)
+			)
+		)
+		(property "LCSC" "C1856484"
 			(at 201.93 71.12 0)
 			(effects
@@
 			)
 		)
+		(property "LCSC" "C1856484"
+			(at 101.6 76.2 0)
+			(effects
+				(font
+					(size 1.27 1.27)
+				)
+				(hide yes)
+			)
+		)
 		(pin "1"
 		)
@@
 			)
 		)
+		(property "LCSC" "C326586"
+			(at 146.05 69.85 0)
+			(effects
+				(font
+					(size 1.27 1.27)
+				)
+				(hide yes)
+			)
+		)
 		(pin "2"
 		)
@@
 			)
 		)
+		(property "LCSC" ""
+			(at 173.99 68.58 0)
+			(effects
+				(font
+					(size 1.27 1.27)
+				)
+			)
+		)
 		(pin "14"
 		)
@@
 			(at 158.75 96.52 0)
 			(effects
+				(font
+					(size 1.27 1.27)
+				)
+				(hide yes)
+			)
+		)
+		(property "LCSC" "C1856484"
+			(at 158.75 96.52 0)
+			(effects
