File: electronics/prototypes/opensync_prototype_4ch/opensync_prototype.kicad_sch (KiCad schematic)
At the start: 0 parts

Commit message: More prototyping
Other:
- added sheet LEDs and Interlock (indicators_and_interlock.kicad_sch)
- sheet Microcontroller and Ext. Clock ports: added ERROR_LED, INTERLOCK_LED, SAFETY_INTERLOCK; removed none
Changed lines of the file:
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@@
+	(wire
+		(pts
+			(xy 78.74 100.33) (xy 105.41 100.33)
+		)
+		(stroke
+			(width 0)
+			(type default)
+		)
+	)
 	(wire
 		(pts
@@
 		(pts
 			(xy 149.86 82.55) (xy 176.53 82.55)
+		)
+		(stroke
+			(width 0)
+			(type default)
+		)
+	)
+	(wire
+		(pts
+			(xy 78.74 105.41) (xy 105.41 105.41)
+		)
+		(stroke
+			(width 0)
+			(type default)
+		)
+	)
+	(wire
+		(pts
+			(xy 78.74 102.87) (xy 105.41 102.87)
 		)
 		(stroke
@@
 			)
 		)
+		(pin "ERROR_LED" output
+			(at 105.41 100.33 180)
+			(effects
+				(font
+					(size 1.27 1.27)
+				)
+				(justify left)
+			)
+		)
+		(pin "INTERLOCK_LED" output
+			(at 105.41 102.87 180)
+			(effects
+				(font
+					(size 1.27 1.27)
+				)
+				(justify left)
+			)
+		)
+		(pin "SAFETY_INTERLOCK" input
+			(at 105.41 105.41 180)
+			(effects
+				(font
+					(size 1.27 1.27)
+				)
+				(justify left)
+			)
+		)
 		(instances
 			(project "opensync_prototype"
@@
 			(project "opensync_prototype"
 				(path "/97d97b34-a2f9-4e5e-9870-299ade25a4f4"
-					(page "7")
+					(page "6")
 				)
 			)
@@
 				)
 			)
+		)
+	)
+	(sheet
+		(at 32.385 97.79)
+		(size 46.355 10.16)
+		(exclude_from_sim no)
+		(in_bom yes)
+		(on_board yes)
+		(dnp no)
+		(fields_autoplaced yes)
+		(stroke
+			(width 0.1524)
+			(type solid)
+		)
+		(fill
+			(color 0 0 0 0.0000)
+		)
+		(property "Sheetname" "LEDs and Interlock"
+			(at 32.385 97.0784 0)
+			(effects
+				(font
+					(size 1.27 1.27)
+				)
+				(justify left bottom)
+			)
+		)
+		(property "Sheetfile" "indicators_and_interlock.kicad_sch"
+			(at 32.385 108.5346 0)
+			(effects
+				(font
+					(size 1.27 1.27)
+				)
+				(justify left top)
+			)
+		)
+		(pin "ERROR_LED" input
+			(at 78.74 100.33 0)
+			(effects
+				(font
+					(size 1.27 1.27)
+				)
+				(justify right)
+			)
+		)
+		(pin "INTERLOCK_LED" input
+			(at 78.74 102.87 0)
+			(effects
+				(font
+					(size 1.27 1.27)
+				)
+				(justify right)
+			)
+		)
+		(pin "SAFETY_INTERLOCK" output
+			(at 78.74 105.41 0)
+			(effects
+				(font
+					(size 1.27 1.27)
+				)
+				(justify right)
+			)
+		)
+		(instances
+			(project "opensync_prototype"
+				(path "/97d97b34-a2f9-4e5e-9870-299ade25a4f4"
+					(page "7")
+				)
+			)
