File: electronics/prototypes/opensync_prototype_4ch/opensync_prototype.kicad_pcb (KiCad board)
At the start: 4 copper layers, 100 x 100 mm, 86 parts, among them J1 61400416121, J12 SM03B-SRSS-TB, J13 61611042121502, J2 61611042121502, J4 61611042121502, J5 61611042121502, J6 61611042121502, J7 61611042121502, SW1 SW_Push, SW2 SW_Push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

Commit message: More prototyping
Parts:
- removed D1, D2: LED, LED_SMD:LED_0603_1608Metric
- added LED1: 5640100132F, 5640100132F:5640100132F, F.Cu at (127.0, 49.6)
- added R15: 120, Resistor_SMD:R_0402_1005Metric, F.Cu at (124.1, 52.1)
- R14: value 100 -> 120
- R9: value 169 -> 120
- moved R9 23.4 mm to (124.1, 49.6), turned to 0 degrees
- moved R14 7.90 mm to (124.1, 54.6), turned to 180 degrees
- moved R8 0.36 mm to (137.6, 91.8), turned to 180 degrees
- moved C22 0.10 mm to (98.4, 82.9)
- turned C18 to 0 degrees
- turned C24 to -90 degrees
- turned C25 to -90 degrees
- turned C26 to -90 degrees
- turned C27 to -90 degrees
- turned C28 to -90 degrees
- turned C29 to -90 degrees
- turned C31 to -90 degrees
- turned R31 to 90 degrees
- turned R35 to 90 degrees
Connections:
- C18 pad 1: VBUS -> GND_BUS
- C18 pad 2: GND_BUS -> VBUS
- C24 pad 1: +3V3 -> GND
- C24 pad 2: GND -> +3V3
- C25 pad 1: +3V3 -> GND
- C25 pad 2: GND -> +3V3
- C26 pad 1: +5V -> GND
- C26 pad 2: GND -> +5V
- C27 pad 1: +5V -> GND
- C27 pad 2: GND -> +5V
- C28 pad 1: +3V3 -> GND
- C28 pad 2: GND -> +3V3
- C29 pad 1: +3V3 -> GND
- C29 pad 2: GND -> +3V3
- C31 pad 1: +5V -> GND
- C31 pad 2: GND -> +5V
- J13 pad 1: /Microcontroller and Ext. Clock/SAFETY_INTERLOCK -> /LEDs and Interlock/SAFETY_INTERLOCK
- R14 pad 1: GND -> Net-(LED1-K_RED)
- R14 pad 2: Net-(D2-K) -> GND
- R31 pad 1: Net-(U6-B) -> Net-(J5-Pad1)
- R31 pad 2: Net-(J5-Pad1) -> Net-(U6-B)
- R35 pad 1: Net-(U8-B) -> Net-(J7-Pad1)
- R35 pad 2: Net-(J7-Pad1) -> Net-(U8-B)
- R8 pad 2: /Microcontroller and Ext. Clock/SAFETY_INTERLOCK -> /LEDs and Interlock/SAFETY_INTERLOCK
- U2 pad 54: /Microcontroller and Ext. Clock/ERROR_LED -> /LEDs and Interlock/ERROR_LED
- U2 pad 55: /Microcontroller and Ext. Clock/SAFETY_INTERLOCK -> /LEDs and Interlock/INTERLOCK_LED
- U2 pad 56: unconnected-(U2-GPIO45_ADC5-Pad56) -> /LEDs and Interlock/SAFETY_INTERLOCK
Routing:
- net /LEDs and Interlock/SAFETY_INTERLOCK: track 0.00 -> 72.2 mm
- net /Microcontroller and Ext. Clock/SAFETY_INTERLOCK: track 71.7 -> 0.00 mm
- net /LEDs and Interlock/ERROR_LED: track 0.00 -> 54.1 mm
- net /LEDs and Interlock/INTERLOCK_LED: track 0.00 -> 50.6 mm
- net /Microcontroller and Ext. Clock/ERROR_LED: track 45.8 -> 0.00 mm
- net GND: track 44.7 -> 47.5 mm, vias 51 -> 54
- net Net-(LED1-K_RED): track 0.00 -> 2.42 mm
- net Net-(LED1-K_YELLOW): track 0.00 -> 2.41 mm
- net Net-(D2-K): track 1.20 -> 0.00 mm
- net Net-(LED1-K_GREEN): track 1.20 -> 2.39 mm
- net +5V: track 23.6 -> 22.6 mm, vias 6 -> 5
Other:
- board text removed: "Error LED Indicator"
- board text removed: "Power LED Indicator"

Commit message: Backup before storm
Routing:
- net /Microcontroller and Ext. Clock/RUN: track 73.6 -> 56.3 mm
- added copper zone on B.Cu, net GND
Changed lines of the file:
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@@
 		(net 44)
 	)
-	(via
+	(via micro
 		(at 95.5 103.6)
 		(size 0.6)
 		(drill 0.3)
-		(layers "F.Cu" "B.Cu")
+		(layers "F.Cu" "In2.Cu")
 		(free yes)
 		(net 44)
 	)
-	(via
+	(via micro
 		(at 132.8 98.55)
 		(size 0.6)
 		(drill 0.3)
-		(layers "F.Cu" "B.Cu")
+		(layers "F.Cu" "In2.Cu")
 		(free yes)
 		(net 44)
 	)
 	(segment
-		(start 134.9 104.5)
-		(end 134.9 111.9)
-		(width 0.1565)
-		(layer "B.Cu")
+		(start 125.3 100.4)
+		(end 98.7 100.4)
+		(width 0.1565)
+		(layer "In2.Cu")
 		(net 44)
 	)
 	(segment
-		(start 134.9 111.9)
-		(end 112.6 111.9)
-		(width 0.1565)
-		(layer "B.Cu")
+		(start 132.119184 100)
+		(end 125.7 100)
+		(width 0.1565)
+		(layer "In2.Cu")
 		(net 44)
 	)
 	(segment
-		(start 132.8 102.4)
-		(end 134.9 104.5)
-		(width 0.1565)
-		(layer "B.Cu")
+		(start 132.8 98.55)
+		(end 132.8 99.319184)
+		(width 0.1565)
+		(layer "In2.Cu")
 		(net 44)
 	)
 	(segment
-		(start 132.8 98.55)
-		(end 132.8 102.4)
-		(width 0.1565)
-		(layer "B.Cu")
+		(start 98.7 100.4)
+		(end 95.5 103.6)
+		(width 0.1565)
+		(layer "In2.Cu")
 		(net 44)
 	)
 	(segment
-		(start 112.6 111.9)
-		(end 104.3 103.6)
-		(width 0.1565)
-		(layer "B.Cu")
+		(start 132.8 99.319184)
+		(end 132.119184 100)
+		(width 0.1565)
+		(layer "In2.Cu")
 		(net 44)
 	)
 	(segment
-		(start 104.3 103.6)
-		(end 95.5 103.6)
-		(width 0.1565)
-		(layer "B.Cu")
+		(start 125.7 100)
+		(end 125.3 100.4)
+		(width 0.1565)
+		(layer "In2.Cu")
 		(net 44)
 	)
@@
 			)
 		)
+	)
+	(zone
+		(net 2)
+		(net_name "GND")
+		(layer "B.Cu")
+		(hatch edge 0.5)
+		(connect_pads
+			(clearance 0.3)
+		)
+		(min_thickness 0.25)
+		(filled_areas_thickness no)
+		(fill yes
+			(thermal_gap 0.5)
+			(thermal_bridge_width 0.5)
+		)
+		(polygon
+			(pts
+				(xy 62 45) (xy 162 45) (xy 163.2 145.5) (xy 62 145)
+			)
+		)
