File: electronics/prototypes/opensync_power_supply_eval/opensync_power_supply_eval.kicad_pcb (KiCad board)
At the start: 2 copper layers, 10 parts, among them J1 61400416121, U1 NCP1117-3.3_SOT223, U3 NXE2S0505MC

Commit message: Finalized dev power PCB
Parts:
- added TP1: TestPoint, TestPoint:TestPoint_Pad_2.0x2.0mm, F.Cu at (106.7, 74.8)
- added TP2: TestPoint, TestPoint:TestPoint_Pad_2.0x2.0mm, F.Cu at (106.7, 82.3)
- added TP3: TestPoint, TestPoint:TestPoint_Pad_2.0x2.0mm, F.Cu at (106.7, 67.3)
- added TP4: TestPoint, TestPoint:TestPoint_Pad_2.0x2.0mm, F.Cu at (87.4, 63.9)
Routing:
- net +5V: track 17.0 -> 20.6 mm
- net GND: track 5.73 -> 7.63 mm, vias 5 -> 6
Other:
- board outline added: 50 x 50 mm
- board text added: "3V"
- board text added: "5V"
- board text added: "GND"
- board text added: "GND_BUS"
