File: electronics/prototypes/opensync_power_supply_eval/opensync_power_supply_eval.kicad_sch (KiCad schematic)
At the start: 10 parts, among them J1 61400416121, U1 NCP1117-3.3_SOT223, U3 NXE2S0505MC

Commit message: More prototyping
Parts:
- renumbered C18 to C1, C20 to C2, C19 to C3, C21 to C4, C22 to C5
Connections:
- net USB_D+: no longer names the net of J1.3 (D+)
- net USB_D-: no longer names the net of J1.2 (D-)
- no-connect marks 0 -> 2
Other:
- company: OpenPIV Consortium -> (none)
- title: OpenSync Power and Data -> (none)
- moved on the sheet: C1, C2, C3, C4, C5, J1, L2, L3, U1, U3

Commit message: Finalized dev power PCB
Parts:
- added TP1, TP2, TP3, TP4: TestPoint, TestPoint:TestPoint_Pad_2.0x2.0mm, symbol Connector:TestPoint
Connections:
- net +3V3: now also TP1.1
- net +5V: now also TP2.1
- net GND: now also TP3.1
- net GND_BUS: now also TP4.1
