File: electronics/prototypes/opensync_prototype_eval/_autosave-prototype_eval.kicad_pcb (KiCad board)
At the start: 2 copper layers, 100 x 100 mm, 60 parts, among them J1 61611042121502, J10 61611042121502, J2 61611042121502, J3 61611042121502, J4 61611042121502, J5 61611042121502, J6 61611042121502, J7 61611042121502, J8 61611042121502, J9 61611042121502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

Commit message: Backup after first PIV experiment
Parts:
- moved R22 175.1 mm to (93.3, 129.0)
- moved J10 172.1 mm to (93.0, 135.0)
- moved C16 35.6 mm to (128.1, 125.0)
- moved R15 35.6 mm to (126.4, 129.2)
- moved C15 35.6 mm to (128.1, 127.7)
- moved R16 35.6 mm to (125.2, 134.4)
- moved U9 35.6 mm to (125.8, 126.3)
- moved J8 28.3 mm to (113.0, 135.0)
Other:
- board size 100 x 100 mm -> 200 x 100 mm
Changed lines of the file:
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@@
 	(footprint "SN74LVC1T45DCKR:SOT65P210X110-6N"
 		(layer "F.Cu")
-		(at 100.45 101.36 -90)
+		(at 125.85 126.35 -90)
 		(property "Reference" "U9"
 			(at -0.56 2.25 180)
@@
 	(footprint "RP2350_80QFN_minimal:C_0402_1005Metric_small_pads"
 		(layer "F.Cu")
-		(at 102.685 100 180)
+		(at 128.085 124.99 180)
 		(descr "Capacitor SMD 0402 (1005 Metric), square (rectangular) end terminal, IPC_7351 nominal, (Body size source: IPC-SM-782 page 76, https://www.pcb-3d.com/wordpress/wp-content/uploads/ipc-sm-782a_amendment_1_and_2.pdf), generated with kicad-footprint-generator")
 		(tags "capacitor")
@@
 	(footprint "RP2350_80QFN_minimal:C_0402_1005Metric_small_pads"
 		(layer "F.Cu")
-		(at 102.7 102.7 180)
+		(at 128.1 127.69 180)
 		(descr "Capacitor SMD 0402 (1005 Metric), square (rectangular) end terminal, IPC_7351 nominal, (Body size source: IPC-SM-782 page 76, https://www.pcb-3d.com/wordpress/wp-content/uploads/ipc-sm-782a_amendment_1_and_2.pdf), generated with kicad-footprint-generator")
 		(tags "capacitor")
@@
 	(footprint "61611042121502:61611042121502"
 		(layer "F.Cu")
-		(at 99.7 110)
+		(at 113 135)
 		(property "Reference" "J8"
 			(at 5.2 -3.065 0)
@@
 	(footprint "61611042121502:61611042121502"
 		(layer "F.Cu")
-		(at 227.34 27.465)
+		(at 93 135)
 		(property "Reference" "J10"
 			(at 8.175 -2.935 0)
@@
 	(footprint "Resistor_SMD:R_0402_1005Metric"
 		(layer "F.Cu")
-		(at 99.8 109.4 -90)
+		(at 125.2 134.39 -90)
 		(descr "Resistor SMD 0402 (1005 Metric), square (rectangular) end terminal, IPC-7351 nominal, (Body size source: IPC-SM-782 page 72, https://www.pcb-3d.com/wordpress/wp-content/uploads/ipc-sm-782a_amendment_1_and_2.pdf), generated with kicad-footprint-generator")
 		(tags "resistor")
@@
 	(footprint "Resistor_SMD:R_0402_1005Metric"
 		(layer "F.Cu")
-		(at 233.345 23.91)
+		(at 93.3 129)
 		(descr "Resistor SMD 0402 (1005 Metric), square (rectangular) end terminal, IPC-7351 nominal, (Body size source: IPC-SM-782 page 72, https://www.pcb-3d.com/wordpress/wp-content/uploads/ipc-sm-782a_amendment_1_and_2.pdf), generated with kicad-footprint-generator")
 		(tags "resistor")
@@
 	(footprint "Resistor_SMD:R_0402_1005Metric"
 		(layer "F.Cu")
-		(at 101.04 104.16 180)
+		(at 126.44 129.15 180)
 		(descr "Resistor SMD 0402 (1005 Metric), square (rectangular) end terminal, IPC-7351 nominal, (Body size source: IPC-SM-782 page 72, https://www.pcb-3d.com/wordpress/wp-content/uploads/ipc-sm-782a_amendment_1_and_2.pdf), generated with kicad-footprint-generator")
 		(tags "resistor")
@@
 	)
 	(gr_line
-		(start 173 138)
-		(end 173 44)
+		(start 273 138)
+		(end 273 44)
 		(stroke
 			(width 0.6)
@@
 	(gr_line
 		(start 76 41)
-		(end 170 41)
+		(end 270 41)
 		(stroke
 			(width 0.6)
@@
 	(gr_line
 		(start 76 141)
-		(end 170 141)
+		(end 270 141)
 		(stroke
 			(width 0.6)
@@
 	)
 	(gr_line
-		(start 73.02132 138.22132)
-		(end 73.02132 44.22132)
+		(start 73 138)
+		(end 73 44)
 		(stroke
 			(width 0.6)
@@
 	)
 	(gr_arc
-		(start 173 138)
-		(mid 172.12132 140.12132)
-		(end 170 141)
+		(start 273 138)
+		(mid 272.12132 140.12132)
+		(end 270 141)
 		(stroke
 			(width 0.6)
@@
 	)
 	(gr_arc
-		(start 170 41)
-		(mid 172.12132 41.87868)
-		(end 173 44)
+		(start 270 41)
+		(mid 272.12132 41.87868)
+		(end 273 44)
 		(stroke
 			(width 0.6)
