File: electronics/prototypes/opensync_prototype_eval/opensync_mounting_holes.kicad_sch (KiCad schematic)
At the start: 4 parts

Commit message: Backup after first PIV experiment
Parts:
- removed H1, H2, H3, H4: MountingHole, MountingHole:MountingHole_3.2mm_M3_ISO7380, symbol Mechanical:MountingHole
