File: electronics/opensync/opensync.kicad_pcb (KiCad board)
At the start: 4 copper layers, 160 x 100 mm, 223 parts, among them J1 SM03B-SRSS-TB, J11 705530001, J12 705530001, J13 MUSBD11130, J14 Barrel_Jack_Switch, J15 Conn_01x02, J16 Conn_01x02, J2 705530001, J3 705530001, J4 705530001, J5 705530001, J6 705530001, J7 705530001, J8 705530001, J9 705530001, SW1 SW_Push, SW2 SW_Push, SW3 2-1825027-0, U1 RP2354_80QFN, U10 SN74LVC2T45DCUR, U11 TPS2116DRL, U12 SN74LVC2T45DCUR, U13 TPS2116DRL, U14 SN74LVC2T45DCUR, U15 TPS2116DRL, U16 SN74LVC2T45DCUR, U17 TPS2116DRL, U2 SN74LVC2T45DCUR, U20 TPD1E05U06DYA, U21 TPD1E05U06DYA, U22 TPD1E05U06DYA, U23 TPD1E05U06DYA, U24 TPD1E05U06DYA, U25 TPD1E05U06DYA, U26 TPD1E05U06DYA, U27 TPD1E05U06DYA, U29 TPD1E05U06DYA, U3 TPS2116DRL, U30 TPD1E05U06DYA, U31 TPS2116DRL, U32 TPS63802DLAR, U33 SN74LVC1G17DCKR, U34 74LVC1G86, U35 SN74LVC1G17DCKR, U36 74LVC1G86, U37 TPS62912, U4 SN74LVC2T45DCUR, U5 TPS2116DRL, U6 SN74LVC2T45DCUR, U7 TPS2116DRL, U8 SN74LVC2T45DCUR, U9 TPS2116DRL, Y1 ABM8-272-T3

Commit message: General revisions
Parts:
- added R62: 10k, Resistor_SMD:R_0402_1005Metric, F.Cu at (78.8, 83.5)
- moved R57 1.69 mm to (79.3, 81.9), turned to 0 degrees
- moved R6 0.99 mm to (79.3, 80.9)
- moved R5 0.86 mm to (79.3, 79.9)
Connections:
- R57 pad 2: /Microcontroller Circuitry/SIG_GATE_INT -> /Microcontroller Circuitry/SIG_INT_TRIG
- U1 pad 1: /Microcontroller Circuitry/SIG_GATE_INT -> /Microcontroller Circuitry/SIG_INT_UNUSED
- U1 pad 78: unconnected-(U1-GPIO1-Pad78) -> /Microcontroller Circuitry/SIG_T0
- U1 pad 79: /Microcontroller Circuitry/SIG_T0 -> /Microcontroller Circuitry/SIG_CLOCK
- U1 pad 80: /Microcontroller Circuitry/SIG_CLOCK -> /Microcontroller Circuitry/SIG_INT_TRIG
Routing:
- net /Microcontroller Circuitry/SIG_INT_TRIG: track 0.00 -> 2.12 mm
- net /Microcontroller Circuitry/SIG_INT_UNUSED: track 0.00 -> 1.38 mm
- net /Microcontroller Circuitry/SIG_GATE_INT: track 1.38 -> 0.00 mm
- net /Microcontroller Circuitry/SIG_CLOCK: track 1.90 -> 3.10 mm
- net /Microcontroller Circuitry/SIG_T0: track 3.44 -> 4.11 mm
- net GND: track 165.7 -> 166.3 mm, vias 190 -> 185
Other:
- board text added: "OpenPIV © 2026 OpenSync v0.4.31"
- board text removed: "OpenPIV © 2026 OpenSync v0.4.29"

Commit message: Updated new design; getting new PCBs
Parts:
- removed C63, C64: 100n, RP2350_80QFN_minimal:C_0402_1005Metric_small_pads
- removed J11, J12: 705530001, 705530001:CONN_705530001_02_MOL
- removed J13: MUSBD11130, MUSBD11130:USB_B_Amphenol_MUSBD11130
- removed R52, R53: 10k, Resistor_SMD:R_0402_1005Metric
- removed R58, R61: 10k, Resistor_SMD:R_0603_1608Metric
- removed R59, R60: 100, Resistor_SMD:R_0603_1608Metric
- removed R75: 301k, Resistor_SMD:R_0402_1005Metric
- removed U29, U30: TPD1E05U06DYA, Diode_SMD:D_SOD-523
- removed U33, U35: SN74LVC1G17DCKR, SN74LVC1G17DCKR:SOT65P210X110-5N
- removed U34, U36: 74LVC1G86, SN74LVC1G17DCKR:SOT65P210X110-5N
- added C58: 1u, Capacitor_SMD:C_0603_1608Metric, F.Cu at (107.2, 120.2)
- added C59: 100p, RP2350_80QFN_minimal:C_0402_1005Metric_small_pads, F.Cu at (108.7, 118.8)
- added C60: 1n, RP2350_80QFN_minimal:C_0402_1005Metric_small_pads, F.Cu at (108.7, 117.8)
- added C61: 100n, RP2350_80QFN_minimal:C_0402_1005Metric_small_pads, F.Cu at (108.7, 116.8)
- added C62: 1u, Capacitor_SMD:C_0603_1608Metric, F.Cu at (108.3, 115.5)
- added C80: 22u, Capacitor_SMD:C_0805_2012Metric, F.Cu at (96.2, 110.0)
- added C81: 22u, Capacitor_SMD:C_0805_2012Metric, F.Cu at (98.3, 110.0)
- added C82: 22u, Capacitor_SMD:C_0805_2012Metric, F.Cu at (93.3, 107.5)
- added D1: ESD701DPYR, ESD701DPYR:X1SON-2_L1.0-W0.6-P0.65-BI, F.Cu at (103.7, 138.0)
- added D11: ESD701DPYR, ESD701DPYR:X1SON-2_L1.0-W0.6-P0.65-BI, F.Cu at (114.7, 138.0)
- added J10: 61729-0010BLF, 61729-0010BLF:AMPHENOL_61729-0010BLF, F.Cu at (115.0, 62.0)
- added J17: 705530001, 705530001:CONN_705530001_02_MOL, F.Cu at (103.0, 140.0)
- added J18: 705530001, 705530001:CONN_705530001_02_MOL, F.Cu at (114.0, 140.0)
- added L5: 7427922808, 7427922808:L0603, F.Cu at (93.1, 110.9)
- added R54: 10k, Resistor_SMD:R_0603_1608Metric, F.Cu at (147.4, 85.3)
- added R55: 5.6k, Resistor_SMD:R_0603_1608Metric, F.Cu at (147.4, 80.5)
- added R72: 10k, Resistor_SMD:R_0402_1005Metric, F.Cu at (111.9, 119.5)
- added R81: 1k, Resistor_SMD:R_0402_1005Metric, F.Cu at (103.5, 133.5)
- added R82: 10k, Resistor_SMD:R_0402_1005Metric, F.Cu at (103.0, 135.0)
- added R83: 1k, Resistor_SMD:R_0402_1005Metric, F.Cu at (114.5, 133.5)
- added R84: 10k, Resistor_SMD:R_0402_1005Metric, F.Cu at (114.0, 135.0)
- added U18: TLV3601DCKR, TLV3601DCKR:SC-70-5_L2.0-W1.3-P0.65-LS2.1-BR, F.Cu at (103.7, 130.0)
- added U19: TLV3601DCKR, TLV3601DCKR:SC-70-5_L2.0-W1.3-P0.65-LS2.1-BR, F.Cu at (114.7, 130.0)
- added U28: DAC8563SDGSR, DAC8563SDGSR:VSSOP-10_L3.0-W3.0-P0.50-LS4.9-BL, F.Cu at (109.9, 122.7)
- C69: value 10u -> 22u
- moved R4 66.0 mm to (131.3, 83.1)
- moved R8 57.8 mm to (127.3, 97.1), turned to -90 degrees
- moved R9 56.1 mm to (127.5, 99.0)
- moved C66 55.8 mm to (116.5, 131.2), turned to 0 degrees
- moved J1 52.4 mm to (90.6, 131.3)
- moved L3 51.3 mm to (89.2, 100.0)
- moved C71 51.3 mm to (96.7, 98.7)
- moved C72 51.3 mm to (98.7, 98.7)
- moved C73 51.3 mm to (95.2, 98.7)
- moved C77 51.3 mm to (95.2, 96.0)
- moved U37 51.3 mm to (93.2, 98.5)
- moved C74 51.3 mm to (93.3, 101.5)
- moved C75 51.3 mm to (93.3, 103.5)
- moved C76 51.3 mm to (93.3, 105.5)
- moved R79 51.3 mm to (93.8, 95.6)
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Connections:
- C67 pad 2: VBUS -> /Power Interface/VDC
- C68 pad 2: /Power Interface/VDC -> VBUS
- C74 pad 2: +3V3 -> +3V3_RAW
- C75 pad 2: +3V3 -> +3V3_RAW
- C76 pad 2: +3V3 -> +3V3_RAW
- L3 pad 2: +3V3 -> +3V3_RAW
- R76 pad 1: Net-(U31-PR1) -> /Power Interface/VDC
- R8 pad 1: /IN_T_INV -> /Input Channels/SIG_TRIG
- R9 pad 1: /IN_T -> /Input Channels/SIG_GATE
- U1 pad 19: /IN_T_INV -> /Input Channels/SIG_TRIG
- U1 pad 20: /IN_T -> /Input Channels/SIG_TRIG
- U1 pad 21: /IN_G_INV -> /Input Channels/SIG_GATE
- U1 pad 22: /IN_G -> /Input Channels/SIG_GATE
- U1 pad 45: unconnected-(U1-GPIO36-Pad45) -> /Microcontroller Circuitry/SENSE_VBUS
- U1 pad 46: unconnected-(U1-GPIO37-Pad46) -> /Input Channels/SPI_SYNC
- U1 pad 47: unconnected-(U1-GPIO38-Pad47) -> /Input Channels/SPI_SCLK
- U1 pad 48: unconnected-(U1-GPIO39-Pad48) -> /Input Channels/SPI_MOSI
- U31 pad 3: /Power Interface/VDC -> VBUS
- U31 pad 4: Net-(U31-PR1) -> GND
- U31 pad 6: VBUS -> /Power Interface/VDC
- U37 pad 3: +3V3 -> +3V3_RAW
Routing:
- net /Input Channels/SPI_SYNC: track 0.00 -> 59.4 mm, vias 0 -> 2
- net /Input Channels/SPI_SCLK: track 0.00 -> 58.6 mm, vias 0 -> 2
- net /Input Channels/SPI_MOSI: track 0.00 -> 57.0 mm, vias 0 -> 2
- net /Input Channels/SIG_TRIG: track 0.00 -> 48.6 mm
- net /IN_T: track 45.1 -> 0.00 mm
- net VBUS: track 23.3 -> 64.5 mm
- net /Input Channels/SIG_GATE: track 0.00 -> 39.2 mm
- net /IN_G: track 38.8 -> 0.00 mm
- net /IN_T_INV: track 38.4 -> 0.00 mm
- net /IN_G_INV: track 30.8 -> 0.00 mm
- net /Microcontroller Circuitry/SENSE_VBUS: track 0.00 -> 24.0 mm, vias 0 -> 2
- net +3V3: track 125.0 -> 109.3 mm
- net /Microcontroller Circuitry/QSPI_SS: track 20.6 -> 6.47 mm
- net /Input Channels/Input Channel 1/SIG_LOGIC: track 0.00 -> 9.68 mm, vias 0 -> 2
- net +3V3_RAW: track 0.00 -> 9.55 mm
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- added copper zone on F.Cu, net +3V3_RAW
Other:
- board text added: "OpenPIV © 2026 OpenSync v0.5.5"
- board text removed: "OpenPIV © 2026 OpenSync v0.4.31"
