File: electronics/opensync/opensync_channel_input.kicad_sch (KiCad schematic)
At the start: 8 parts, among them J11 705530001, U29 TPD1E05U06DYA, U33 SN74LVC1G17DCKR, U34 74LVC1G86

Commit message: Updated new design; getting new PCBs
Parts:
- removed C64: 100n, RP2350_80QFN_minimal:C_0402_1005Metric_small_pads, symbol Device:C
- removed U29: TPD1E05U06DYA, Diode_SMD:D_SOD-523, symbol Power_Protection:TPD1E05U06DYA
- removed U33: SN74LVC1G17DCKR, SN74LVC1G17DCKR:SOT65P210X110-5N, symbol SN74LVC1G17DCKR:SN74LVC1G17DCKR
- removed U34: 74LVC1G86, SN74LVC1G17DCKR:SOT65P210X110-5N, symbol 74xGxx:74LVC1G86
- added D1: ESD701DPYR, ESD701DPYR:X1SON-2_L1.0-W0.6-P0.65-BI, symbol ESD701DPYR:ESD701DPYR
- added U18: TLV3601DCKR, TLV3601DCKR:SC-70-5_L2.0-W1.3-P0.65-LS2.1-BR, symbol TLV3601DCKR:TLV3601DCKR
- C65: renamed from C63; Description_1 (none) -> 100nF ceramic MLCC, 50V, ±10%, X7R, 0402 (1005 metric); operating_temp_max (none) -> 125 C; operating_temp_min (none) -> -55 C; polarity (none) -> Non-polarized
- J17: renamed from J11; LCSC (none) -> C564143
- R81: renamed from R59; value 100 -> 1k; footprint Resistor_SMD:R_0603_1608Metric -> Resistor_SMD:R_0402_1005Metric; Description_1 (none) -> 1kΩ ±1% thick film resistor, 200mW, 50V, 0402 (1005 metric); LCSC C844917 -> C313354; manufacturer_pn CRCW0603100RFKEA -> CRCW04021K00FKEDHP; package 0603 (1608 metric) -> 0402 (1005 metric); power 100mW -> 200mW; resistance 100Ω -> 1kΩ; voltage 75V -> 50V
- R82: renamed from R58; footprint Resistor_SMD:R_0603_1608Metric -> Resistor_SMD:R_0402_1005Metric; Description_1 (none) -> 10kΩ ±1% thick film resistor, 63mW, 50V, 0402 (1005 metric); LCSC C844918 -> C71617; manufacturer_pn CRCW060310K0FKEA -> CRCW040210K0FKED; package 0603 (1608 metric) -> 0402 (1005 metric); power 100mW -> 63mW; voltage 75V -> 50V
Connections:
- net +3V3: now also U18.5 (VCC)
- net GND: now also R81.2, D1.2, U18.2 (VEE); no longer R82.2
- net SIG_TRIG: now also U18.1 (OUT)
- net at R82.1: now also R81.1, U18.4 (IN-); no longer R81.2
- net at J17.1: now also R82.2, D1.1; no longer R81.1
- new net SIG_LOGIC: U18.3 (IN+)
Other:
- moved on the sheet: C65, R81, R82
