File: electronics/opensync/opensync_channel_output.kicad_sch (KiCad schematic)
At the start: 14 parts, among them J2 705530001, U2 SN74LVC2T45DCUR, U20 TPD1E05U06DYA, U3 TPS2116DRL

Commit message: Updated new design; getting new PCBs
Parts:
- C18, C19: Description_1 (none) -> 1uF automotive ceramic MLCC, 25V, +/-10%, X7R, 0603; operating_temp_max (none) -> 125 C; operating_temp_min (none) -> -55 C; polarity (none) -> Non-polarized; tolerance ±10% -> +/-10%
- C20, C22: Description_1 (none) -> 100nF ceramic MLCC, 50V, ±10%, X7R, 0402 (1005 metric); operating_temp_max (none) -> 125 C; operating_temp_min (none) -> -55 C; polarity (none) -> Non-polarized
- C21: Description_1 (none) -> 22uF SMD aluminum electrolytic, 10V, +/-20%, WCAP-ASLL, dia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; dielectric (none) -> Aluminum oxide; impedance (none) -> 1.35 ohm max at 100kHz, 20 C; lifetime 2000hrs@105℃ -> 2000h at 105 C; material Aluminum Electrolytic -> Aluminum electrolytic; operating_temp_max +105C -> 105 C; operating_temp_min -55C -> -55 C; package SMD, D4x5.5mm -> SMD, D4xL5.5mm; ripple_current 58.5mA@120Hz -> 90mA at 100kHz, 105 C; tolerance ±20% -> +/-20%
- J2: LCSC (none) -> C564143
- R12, R15: Description_1 (none) -> 10kΩ ±1% thick film resistor, 63mW, 0402 (1005 metric)
- R13: Description_1 (none) -> 47kΩ ±1% thick film resistor, 62.5mW, 0402 (1005 metric)
- R14: Description_1 (none) -> 39 ohm +/-1% 0.25 W at 70 C, 150 V limiting element voltage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; LCSC C2105598 -> C544038; manufacturer Vishay Intertech -> Panasonic; manufacturer_pn RCS060339R0FKEA -> ERJUP3F39R0V; operating_temp_max +155C -> 155 C; operating_temp_min -55C -> -55 C; power 250mW -> 0.25 W; resistance 39Ω -> 39 ohm; technology Thick Film Resistor -> Anti-surge sulfur-resistant thick film; temp_coefficient ±100ppm/℃ -> +/-100 ppm/C; tolerance ±1% -> +/-1%; voltage 75V -> 150 V
- R16: Description_1 (none) -> 10kΩ ±1% thick film resistor, 100mW, 0603 (1608 metric)
