File: electronics/opensync/opensync_interface_power.kicad_sch (KiCad schematic)
At the start: 27 parts, among them J14 Barrel_Jack_Switch, J15 Conn_01x02, J16 Conn_01x02, U31 TPS2116DRL, U32 TPS63802DLAR, U37 TPS62912

Commit message: Updated new design; getting new PCBs
Parts:
- removed R75: 301k, Resistor_SMD:R_0402_1005Metric, symbol Device:R
- added C80, C81, C82: 22u, Capacitor_SMD:C_0805_2012Metric, symbol Device:C
- added L5: 7427922808, 7427922808:L0603, symbol 7427922808:7427922808
- C67, C68: Description_1 (none) -> 1uF automotive ceramic MLCC, 25V, +/-10%, X7R, 0603; operating_temp_max (none) -> 125 C; operating_temp_min (none) -> -55 C; polarity (none) -> Non-polarized; tolerance ±10% -> +/-10%
- C69: value 10u -> 22u; Description_1 (none) -> 22uF ceramic MLCC, 10V, ±20%, X7S, 0805 (2012 metric); LCSC C342722 -> C342717; capacitance 10uF -> 22uF; dielectric X5R -> X7S; manufacturer_pn C2012X5R1V106KT000E -> C2012X7S1A226MT000E; operating_temp_max (none) -> 125 C; operating_temp_min (none) -> -55 C; polarity (none) -> Non-polarized; tolerance ±10% -> ±20%; voltage 35V -> 10V
- C70, C78: Description_1 (none) -> 22uF ceramic MLCC, 10V, ±20%, X7S, 0805 (2012 metric); LCSC C338080 -> C342717; dielectric X5R -> X7S; manufacturer_pn C2012X5R1V226MT000E -> C2012X7S1A226MT000E; operating_temp_max (none) -> 125 C; operating_temp_min (none) -> -55 C; polarity (none) -> Non-polarized; voltage 35V -> 10V
- C71, C72: Description_1 (none) -> 10uF ceramic MLCC, 35V, ±10%, X5R, 0805 (2012 metric); operating_temp_max (none) -> 85 C; operating_temp_min (none) -> -55 C; polarity (none) -> Non-polarized
- C73: Description_1 (none) -> 2.2nF automotive ceramic MLCC, 50V, +/-10%, X7R, 0402; operating_temp_max (none) -> 125 C; operating_temp_min (none) -> -55 C; polarity (none) -> Non-polarized; tolerance ±10% -> +/-10%
- C74, C75, C76: Description_1 (none) -> 22uF ceramic MLCC, 10V, ±20%, X7S, 0805 (2012 metric); LCSC C338078 -> C342717; dielectric X5R -> X7S; manufacturer_pn C2012X5R1E226MT000E -> C2012X7S1A226MT000E; operating_temp_max (none) -> 125 C; operating_temp_min (none) -> -55 C; polarity (none) -> Non-polarized; voltage 25V -> 10V
- C77: Description_1 (none) -> 470nF automotive ceramic MLCC, 16V, +/-10%, X7S, 0402; operating_temp_max (none) -> 125 C; operating_temp_min (none) -> -55 C; polarity (none) -> Non-polarized; tolerance ±10% -> +/-10%
- C79: Description_1 (none) -> 100nF ceramic MLCC, 50V, ±10%, X7R, 0402 (1005 metric); operating_temp_max (none) -> 125 C; operating_temp_min (none) -> -55 C; polarity (none) -> Non-polarized
- J15, J16: LCSC (none) -> C127361
- R76: Description_1 (none) -> 100kΩ ±1% thick film resistor, 63mW, 0402 (1005 metric)
- R77: Description_1 (none) -> 806 kohm +/-1%, 0402 thick film resistor, 0.063 W at 70 C, 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; manufacturer Vishay Intertech -> Vishay; operating_temp_max +155C -> 155 C; operating_temp_min -55C -> -55 C; power 62.5mW -> 0.063 W; resistance 806kΩ -> 806 kohm; technology Thick Film Resistor -> Thick film; temp_coefficient ±100ppm/℃ -> +/-100 ppm/C; tolerance ±1% -> +/-1%; voltage 75V -> 50 V
- R78: Description_1 (none) -> 91 kohm +/-1%, 0402 thick film resistor, 0.063 W at 70 C, 5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; manufacturer Vishay Intertech -> Vishay; operating_temp_max +155C -> 155 C; operating_temp_min -55C -> -55 C; power 62.5mW -> 0.063 W; resistance 91kΩ -> 91 kohm; technology Thick Film Resistor -> Thick film; temp_coefficient ±100ppm/℃ -> +/-100 ppm/C; tolerance ±1% -> +/-1%; voltage 50V -> 50 V
- R79: Description_1 (none) -> 4.99 kohm +/-1%, 0402 thick film resistor, 0.063 W at 70 C,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; manufacturer Vishay Intertech -> Vishay; operating_temp_max +155C -> 155 C; operating_temp_min -55C -> -55 C; power 62.5mW -> 0.063 W; resistance 4.99kΩ -> 4.99 kohm; technology Thick Film Resistor -> Thick film; temp_coefficient ±100ppm/℃ -> +/-100 ppm/C; tolerance ±1% -> +/-1%; voltage (none) -> 50 V
- R80: Description_1 (none) -> 15.6 kohm +/-0.1%, 0402 thin film resistor, 0.1 W at 70 C, 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; manufacturer Vishay Intertech -> Vishay; operating_temp_max +155C -> 155 C; operating_temp_min -55C -> -55 C; power 100mW -> 0.1 W; resistance 15.6kΩ -> 15.6 kohm; technology Thin Film Resistor -> Thin film; temp_coefficient ±25ppm/℃ -> +/-25 ppm/C; tolerance ±0.1% -> +/-0.1%; voltage 50V -> 50 V
Connections:
- net +3V3: now also C80.2, C81.2, L5.2; no longer C74.2, C75.2, C76.2, L3.2, U37.3 (VO)
- net GND: now also U31.4 (PR1), C80.1, C81.1, C82.1
- net VBUS: now also C68.2, U31.3 (VIN1); no longer C67.2, U31.6 (VIN2)
- net VDC: now also C67.2, R76.1, U31.6 (VIN2); no longer C68.2, U31.3 (VIN1)
- new net +3V3_RAW: C74.2, C75.2, C76.2, C82.2, L3.2, L5.1, U37.3 (VO)
Other:
- moved on the sheet: R76, R77, R78
