File: electronics/opensync/opensync_interface_usb.kicad_sch (KiCad schematic)
At the start: 4 parts, among them J13 MUSBD11130

Commit message: Updated new design; getting new PCBs
Parts:
- removed J13: MUSBD11130, MUSBD11130:USB_B_Amphenol_MUSBD11130, symbol MUSBD11130:MUSBD11130
- added J10: 61729-0010BLF, 61729-0010BLF:AMPHENOL_61729-0010BLF, symbol 61729-0010BLF:61729-0010BLF
- added R54: 10k, Resistor_SMD:R_0603_1608Metric, symbol Device:R
- added R55: 5.6k, Resistor_SMD:R_0603_1608Metric, symbol Device:R
Connections:
- net GND: now also J10.4 (GND), J10.SH1 (SHIELD), J10.SH2 (SHIELD), R54.2
- net VBUS: now also R55.1
- net VBUS_RAW: now also J10.1 (VCC)
- net at D14.3 (I/O_1), L4.2: now also J10.3 (D+)
- net at D14.4 (I/O_2), L4.3: now also J10.2 (D-)
- new net SENSE_VBUS: R54.1, R55.2
