File: electronics/opensync/opensync_microcontroller.kicad_sch (KiCad schematic)
At the start: 37 parts, among them J1 SM03B-SRSS-TB, SW1 SW_Push, SW2 SW_Push, U1 RP2354_80QFN, Y1 ABM8-272-T3

Commit message: General revisions
Parts:
- added R62: 10k, Resistor_SMD:R_0402_1005Metric, symbol Device:R
Connections:
- net GND: now also R62.1
- net SIG_CLOCK: now also U1.79 (GPIO2); no longer U1.80 (GPIO3)
- net SIG_T0: now also U1.78 (GPIO1); no longer U1.79 (GPIO2)
- net SIG_GATE_INT renamed SIG_INT_TRIG
- net SIG_INT_TRIG: now also U1.80 (GPIO3); no longer U1.1 (GPIO4)
- new net SIG_INT_UNUSED: R62.2, U1.1 (GPIO4)
- no-connect marks 18 -> 17
Other:
- moved on the sheet: R5, R57, R6

Commit message: Updated new design; getting new PCBs
Parts:
- removed R53, R9: 10k, Resistor_SMD:R_0402_1005Metric, symbol Device:R
- C1, C4, C5: Description_1 (none) -> 4.7uF ceramic MLCC, 10V, ±10%, X5R, 0402 (1005 metric); operating_temp_max (none) -> 85 C; operating_temp_min (none) -> -55 C; polarity (none) -> Non-polarized
- C10, C11, C12, C13, C14, C15, C16, C17, C6, C7, C8, C9: Description_1 (none) -> 100nF ceramic MLCC, 50V, ±10%, X7R, 0402 (1005 metric); operating_temp_max (none) -> 125 C; operating_temp_min (none) -> -55 C; polarity (none) -> Non-polarized
- C2, C3: Description_1 (none) -> 15pF ceramic MLCC, 50V, ±5%, C0G, 0402 (1005 metric); operating_temp_max (none) -> 125 C; operating_temp_min (none) -> -55 C; polarity (none) -> Non-polarized
- R1: Description_1 (none) -> 33Ω ±1% thick film resistor, 62.5mW, 0402 (1005 metric); voltage (none) -> 50 V
- R10, R11: Description_1 (none) -> 27 ohm +/-1%, 0402 thick film resistor, 0.063 W at 70 C, 50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; manufacturer Vishay Intertech -> Vishay; operating_temp_max (none) -> 155 C; operating_temp_min (none) -> -55 C; power 62.5mW -> 0.063 W; resistance 27Ω -> 27 ohm; technology Thick Film Resistor -> Thick film; temp_coefficient ±100ppm/℃ -> +/-100 ppm/C; tolerance ±1% -> +/-1%; voltage (none) -> 50 V
- R2, R3, R4: Description_1 (none) -> 1kΩ ±1% thick film resistor, 200mW, 0402 (1005 metric)
- R5, R57, R6, R62, R7, R8: Description_1 (none) -> 10kΩ ±1% thick film resistor, 63mW, 0402 (1005 metric)
- R9: renamed from R52; Description_1 (none) -> 10kΩ ±1% thick film resistor, 63mW, 0402 (1005 metric)
Connections:
- net IN_GATE_I is gone; now on net IN_GATE: R9.1, U1.21 (GPIO21)
- net IN_TRIG_I is gone; now on net IN_TRIG: R8.1, U1.19 (GPIO19)
- net SENSE_VBUS: now reaches U1.45 (GPIO36)
- net SCPI_SYNC: now reaches U1.46 (GPIO37)
- net SCPI_SCLK: now reaches U1.47 (GPIO38)
- net SCPI_MOSI: now reaches U1.48 (GPIO39)
- no-connect marks 17 -> 13
Other:
- moved on the sheet: R8, R9
