File: electronics/opensync/opensync_panel_indicator.kicad_sch (KiCad schematic)
At the start: 23 parts, among them SW3 2-1825027-0

Commit message: Updated new design; getting new PCBs
Parts:
- R63, R64, R65, R66, R67, R68, R69, R70, R71, R73, R74: Description_1 (none) -> 470Ω ±1% thick film resistor, 100mW, 0603 (1608 metric)
